File: SMeter_RevA.sch (EAGLE design)
At the start: 46 parts, among them IC1 AD8307, IC2 AD603, IC3 TL081

Commit message: Revision B finalized
Parts:
- C2, C3: value 33u -> 47u
- L2, L3: value (none) -> 100uH
Changed lines of the file:
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@@
 <part name="GND1" library="00Supply" deviceset="GND" device=""/>
 <part name="C1" library="00Capacitor" deviceset="C" device="C0805" value="18p"/>
-<part name="C2" library="00Capacitor" deviceset="C_POLARIZED" device="SMC_B" value="33u"/>
-<part name="C3" library="00Capacitor" deviceset="C_POLARIZED" device="SMC_B" value="33u"/>
+<part name="C2" library="00Capacitor" deviceset="C_POLARIZED" device="SMC_B" value="47u"/>
+<part name="C3" library="00Capacitor" deviceset="C_POLARIZED" device="SMC_B" value="47u"/>
 <part name="IC2" library="00Amplifier" deviceset="AD603" device=""/>
 <part name="R1" library="00Resistor" deviceset="RESISTOR" device="R0805" value="100k"/>
@@
 <part name="L1" library="00Inductor" deviceset="INDUCTOR" device="0805" value="880n"/>
 <part name="R7" library="00Resistor" deviceset="RESISTOR" device="R0805" value="15k"/>
-<part name="L2" library="00Inductor" deviceset="INDUCTOR" device="LPS4018"/>
-<part name="L3" library="00Inductor" deviceset="INDUCTOR" device="LPS4018"/>
+<part name="L2" library="00Inductor" deviceset="INDUCTOR" device="LPS4018" value="100uH"/>
+<part name="L3" library="00Inductor" deviceset="INDUCTOR" device="LPS4018" value="100uH"/>
 <part name="P+3" library="00Supply" deviceset="+5V" device=""/>
 <part name="P-2" library="00Supply" deviceset="-5V" device=""/>
